File: magnetic_keyboard_meishi.kicad_sch (KiCad schematic)
At the start: 0 parts

Commit message: DRV5055の追加
Parts:
- added U1, U2, U3, U4, U5, U6, U7, U8: DRV5055A4xDBZxQ1, Package_TO_SOT_SMD:SOT-23, symbol Sensor_Magnetic:DRV5055A4xDBZxQ1
